File: hardware/can-bb.brd (EAGLE design)
At the start: 36 x 16 mm, 10 parts, among them J1 MF-CON-2.54mm-01x02, J2 EZMATE-5, J3 RJ45-8PTH, J4 RJ45-8PTH, J5 EZMATE-5

Commit message: hw: 2021: add few notes
Parts:
- R5: value 10k -> 22k
Changed lines of the file:
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@@
 <attribute name="VALUE" x="19.06" y="8.635" size="1.27" layer="27" rot="R270"/>
 </element>
-<element name="R5" library="balto" package="0603" value="10k" x="17.2" y="9.2" smashed="yes" rot="R90">
+<element name="R5" library="balto" package="0603" value="22k" x="17.2" y="9.2" smashed="yes" rot="R90">
 <attribute name="NAME" x="16.438" y="7.676" size="1.27" layer="25" rot="R90"/>
 <attribute name="VALUE" x="19.232" y="7.676" size="1.27" layer="27" rot="R90"/>
