File: hardware/can-bb.sch (EAGLE design)
At the start: 9 parts, among them J1 MF-CON-2.54mm-01x02, J2 EZMATE-5, J3 RJ45-8PTH, J4 RJ45-8PTH, J5 EZMATE-5

Commit message: hw: 2021: add few notes
Parts:
- R5: value 10k -> 22k
Changed lines of the file:
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@@
 <part name="FRAME1" library="frames" library_urn="urn:adsk.eagle:library:229" deviceset="A5L-LOC" device=""/>
 <part name="J3" library="balto" deviceset="RJ45-8" device="PTH"/>
-<part name="R5" library="balto" deviceset="R" device="0603" value="10k"/>
+<part name="R5" library="balto" deviceset="R" device="0603" value="22k"/>
 <part name="LED4" library="led" library_urn="urn:adsk.eagle:library:259" deviceset="LED" device="CHIPLED_0603" package3d_urn="urn:adsk.eagle:package:15822/2"/>
 <part name="GND1" library="supply1" deviceset="GND" device=""/>
