File: hardware/open-usb-can-2021.brd (EAGLE design)
At the start: 53.6 x 18.2 mm, 36 parts, among them J1 MF-CON-2.54mm-01x02, J2 EZMATE-3, J3 RJ45-8PTH, J4 EZMATE-4, J6 EZMATE-5, Q1 16MHz, U1 MCP2515-I/P, U2 ATMEGA32U2-AU, U5 MAX3051

Commit message: hw: 2021: add few notes
Parts:
- R29, R30, R4: value 5k6 -> 1k
- R36: value 100k -> 0
- R5: value 10k -> 22k
Changed lines of the file:
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@@
 <attribute name="VALUE" x="5.565" y="7.895" size="1.27" layer="27"/>
 </element>
-<element name="R29" library="balto" package="0402" value="5k6" x="4.8" y="16.2" smashed="yes">
+<element name="R29" library="balto" package="0402" value="1k" x="4.8" y="16.2" smashed="yes">
 <attribute name="NAME" x="3.276" y="16.962" size="1.27" layer="25"/>
 <attribute name="VALUE" x="3.276" y="14.168" size="1.27" layer="27"/>
@@
 <attribute name="VALUE" x="5.565" y="6.695" size="1.27" layer="27"/>
 </element>
-<element name="R30" library="balto" package="0402" value="5k6" x="5" y="2.6" smashed="yes">
+<element name="R30" library="balto" package="0402" value="1k" x="5" y="2.6" smashed="yes">
 <attribute name="NAME" x="3.476" y="3.362" size="1.27" layer="25"/>
 <attribute name="VALUE" x="3.476" y="0.568" size="1.27" layer="27"/>
@@
 <attribute name="VALUE" x="36.26" y="3.035" size="1.27" layer="27" rot="R270"/>
 </element>
-<element name="R36" library="balto" package="0603" value="100k" x="39" y="9.8" smashed="yes">
+<element name="R36" library="balto" package="0603" value="0" x="39" y="9.8" smashed="yes">
 <attribute name="NAME" x="37.476" y="10.562" size="1.27" layer="25"/>
 <attribute name="VALUE" x="37.476" y="7.768" size="1.27" layer="27"/>
 </element>
-<element name="R4" library="balto" package="0402" value="5k6" x="4.8" y="15" smashed="yes">
+<element name="R4" library="balto" package="0402" value="1k" x="4.8" y="15" smashed="yes">
 <attribute name="NAME" x="3.276" y="15.762" size="1.27" layer="25"/>
 <attribute name="VALUE" x="3.276" y="12.968" size="1.27" layer="27"/>
 </element>
-<element name="R5" library="balto" package="0603" value="10k" x="39" y="12.4" smashed="yes">
+<element name="R5" library="balto" package="0603" value="22k" x="39" y="12.4" smashed="yes">
 <attribute name="NAME" x="37.476" y="13.162" size="1.27" layer="25"/>
 <attribute name="VALUE" x="37.476" y="10.368" size="1.27" layer="27"/>
