File: hardware/open-usb-can-2021.sch (EAGLE design)
At the start: 35 parts, among them J1 MF-CON-2.54mm-01x02, J2 EZMATE-3, J3 RJ45-8PTH, J4 EZMATE-4, J6 EZMATE-5, Q1 16MHz, U1 MCP2515-I/P, U2 ATMEGA32U2-AU, U5 MAX3051

Commit message: hw: 2021: add few notes
Parts:
- R29, R30, R4: value 5k6 -> 1k
- R36: value 100k -> 0
- R5: value 10k -> 22k
Other:
- note added: "TODO: - connect INT - fix xcvr AGND - add xcvr cap"
Changed lines of the file:
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@@
 <part name="GND39" library="supply1" deviceset="GND" device=""/>
 <part name="+3V9" library="supply1" deviceset="+3V3" device=""/>
-<part name="R36" library="balto" deviceset="R" device="0603" value="100k"/>
+<part name="R36" library="balto" deviceset="R" device="0603" value="0"/>
 <part name="R2" library="balto" deviceset="R" device="0603" value="22"/>
 <part name="R3" library="balto" deviceset="R" device="0603" value="22"/>
@@
 <part name="GND6" library="supply1" deviceset="GND" device=""/>
 <part name="+3V3" library="supply1" deviceset="+3V3" device=""/>
-<part name="R29" library="balto" deviceset="R" device="0402" value="5k6"/>
+<part name="R29" library="balto" deviceset="R" device="0402" value="1k"/>
 <part name="LED2" library="led" library_urn="urn:adsk.eagle:library:259" deviceset="LED" device="CHIPLED_0603" package3d_urn="urn:adsk.eagle:package:15822/2"/>
 <part name="LED3" library="led" library_urn="urn:adsk.eagle:library:259" deviceset="LED" device="CHIPLED_0603" package3d_urn="urn:adsk.eagle:package:15822/2"/>
-<part name="R30" library="balto" deviceset="R" device="0402" value="5k6"/>
+<part name="R30" library="balto" deviceset="R" device="0402" value="1k"/>
 <part name="+3V4" library="supply1" deviceset="+3V3" device=""/>
 <part name="GND7" library="supply1" deviceset="GND" device=""/>
-<part name="R4" library="balto" deviceset="R" device="0402" value="5k6"/>
+<part name="R4" library="balto" deviceset="R" device="0402" value="1k"/>
 <part name="LED1" library="led" library_urn="urn:adsk.eagle:library:259" deviceset="LED" device="CHIPLED_0603" package3d_urn="urn:adsk.eagle:package:15822/2"/>
 <part name="C4" library="balto" deviceset="C" device="0402" value="100n"/>
@@
 <part name="+3V2" library="supply1" deviceset="+3V3" device=""/>
 <part name="J1" library="MF_Connectors" deviceset="CON_01X02" device="_PTH_2.54MM" value="MF-CON-2.54mm-01x02"/>
-<part name="R5" library="balto" deviceset="R" device="0603" value="10k"/>
+<part name="R5" library="balto" deviceset="R" device="0603" value="22k"/>
 <part name="LED4" library="led" library_urn="urn:adsk.eagle:library:259" deviceset="LED" device="CHIPLED_0603" package3d_urn="urn:adsk.eagle:package:15822/2"/>
 <part name="GND1" library="supply1" deviceset="GND" device=""/>
@@
 <text x="5.08" y="116.84" size="5.08" layer="97">CAN XCVR</text>
 <text x="236.22" y="63.5" size="5.08" layer="97">HWB</text>
+<text x="63.5" y="88.9" size="1.778" layer="97">TODO:
+- connect INT
+- fix xcvr AGND
+- add xcvr cap</text>
 </plain>
 <instances>
@@
 </drawing>
 <compatibility>
+<note version="6.3" minversion="6.2.2" severity="warning">
+Since Version 6.2.2 text objects can contain more than one line,
+which will not be processed correctly with this version.
+</note>
 <note version="8.2" severity="warning">
 Since Version 8.2, EAGLE supports online libraries. The ids
